File: LVC/LVC.kicad_sch (KiCad schematic)
At the start: 5 parts, among them U1 TL431DBZ

Commit message: Testing Schematics Added
Added the schematics for the circuits used during testing. This is synced up with documentation of such tests in Bear.
Parts:
- removed F1: Fuse, symbol Device:Fuse
- removed R1: POT, symbol Device:R_Variable_US
- removed R2: 10kΩ, symbol Device:R_US
- removed R3: 6kΩ, symbol Device:R_US
- removed U1: TL431DBZ, Package_TO_SOT_SMD:SOT-23, symbol Reference_Voltage:TL431DBZ

Commit message: Refining Schematics
Refined the visuals of all the schematics to remove values from components. Also removed a redundant schematic.
Parts:
- added Q1: IRF9540N, Package_TO_SOT_THT:TO-220-3_Vertical, symbol Transistor_FET:IRF9540N
- added R10, R4, R5, R6, R7, R8, R9: R_US, symbol Device:R_US
- added U2: TL431DBZ, Package_TO_SOT_SMD:SOT-23, symbol Reference_Voltage:TL431DBZ
- added U3: LM393, symbol Comparator:LM393
Connections:
- new net: Q1.1 (G), R9.2
- new net: R7.2, R8.1
- new net: R6.2, U2.1 (K), U3.3 (+)
- new net: R4.2, R5.1, U2.2 (REF)
- new net GND: R5.2, R8.2, U2.3 (A)
- new net VCC: Q1.2 (D), R4.1, R6.1, R7.1, R9.1

Commit message: LVC Prototype
Initial design concept created. Testing in progress.
Parts:
- added D1: LED, symbol Device:LED
- added R6, R7: R_US, symbol Device:R_US
- U1: renamed from U2; value TL431DBZ -> TL431A
- renumbered R4 to R1, R5 to R2, R6 to R3, R7 to R4, R8 to R5, R10 to R8
Connections:
- net GND: now also R7.2
- net VCC: now also R6.1; no longer R4.1
- net at Q1.1 (G), R9.2: now also R8.2, U3.1
- net at R4.2, R5.1: now also R8.1, U3.3 (+)
- net at U3.2 (-): now also R6.2, R7.1
- new net: D1.1 (K), R4.1, U1.1 (K)
- new net: D1.2 (A), R3.2
Other:
- moved on the sheet: Q1, R1, R2, R4, R5, R8, U1, U3A
